File: OpenROV Controller.brd (EAGLE design)
At the start: 150 x 80 mm, 183 parts, among them J1 SSW-108-01-G-D, J18 SSW-103-01-G-D, J19 SSW-103-01-G-D, J2 SSW-108-01-G-D, J20 TSW-103-07-G-T, J21 TSW-103-07-G-T, J3 SSW-108-01-G-D, J4 SSW-108-01-G-D, J5 FCI 10090096-P254, J6 Samtec DW-23-11-G-D-630, Q1 SI4485, Q2 DMN65D8L, Q3 SI4425, Q4 IRLML6346TR, Q5 IRLML6346TR, Q6 IRLML6346TR, Q7 IRLML6346TR, Q8 FDV301N, Q9 FDV301N, U1 INA199A2, U10 INA199A2, U11 INA199A2, U2 INA199A2, U3 INA199A2, U4 LM25011, U5 TLV1117LV33, U6 ATMEGA2560-16AU, U7 TXB0108SSOP-20, U8 CAT24C256WI-G, U9 INA199A2, X1 16 MHz

Commit message: Checkin of the 2.7 schematics
Parts:
- removed R15: 0.075 1%, Walts_Generic_Parts:R1210
- added C39, C40, C41: 220 uF 35V Low-Impedance, Walts_Generic_Parts:NICHICON_10MM
- added C42, C44: 1 uF 25V X7R, Walts_Generic_Parts:R0603
- added C43: 0.1 uF, Walts_Generic_Parts:R0603
- added U$1: (no value), OpenROV General Library:OROV-LOGO-2.00
- added U$2: (no value), OpenROV General Library:CC-LOGO-1
- added U12: TCR2EF33, Walts Power Supply Components:SOT23-5L
- C10: value 1 uF 50V X5R -> 3900 pF 25V NP0; device Walts_Generic_Parts:R0805 -> Walts_Generic_Parts:R0603
- C11: value 1000 pF 50V X7R -> 3900 pF 25V NP0
- C13, C14: value 10 uF 10V X5R -> 22 uF 10V X5R
- C16: value 10 uF 10V X5R -> 10 uF 25V X5R
- C34: value 220 uF 6.3V -> 220 uF 10V; device Walts_Generic_Parts:KEMET_B-CAPACITOR -> Walts_Generic_Parts:NICHICON_8MM
- C35: value DNP -> 10 uF 25V X5R
- C8, C9: value 1 uF 50V X5R -> 10 uF 25V X5R
- D3: value SMAJ22A -> SMAJ18A
- D6: value CDBA340 -> SMAJ15A
- F1: value 1.95A / 1.1A -> 2.0A / 4.0A 24V; device Walts_Generic_Parts:R1812 -> Walts_Generic_Parts:R2920
- J14: device OpenROV General Library:ESC-PADS-.156-ALT_SILK -> OpenROV General Library:AFRO-ESC-12/20A-ESC1
- J15: device OpenROV General Library:ESC-PADS-.156-ALT_SILK -> OpenROV General Library:AFRO-ESC-12/20A-ESC2
- J16: device OpenROV General Library:ESC-PADS-.156-ALT_SILK -> OpenROV General Library:AFRO-ESC-12/20A-ESC3
- J18, J19: value SSW-103-01-G-D -> Sullins PRPC003DFAN-RC
- L1: value MSS1048-153MLB -> 15 uH 4A; device OpenROV Controller 2.5:MSS1048 -> Walts_Generic_Parts:INDUCTOR_BOURNS_12X0
- LED1, LED6: value Green -> GREEN
- LED7, LED8: value Yellow -> YELLOW
- Q3: value SI4425 -> SI4459ADY
- R13: value 10K -> 100K
- R14: value 133K 1% -> 13.0K 1%
- R16: value 9.76K 1% -> 45.3K 1%
- R24, R25, R26, R27, R28, R29, R30, R31, R32, R33, R34, R35: device Walts_Generic_Parts:R0603 -> Walts_Generic_Parts:R0805
- R67: value 0 -> 0 (Jumper)
- U4: value LM25011 -> Richtek RT8250; device OpenROV Controller 2.5:VSSOP-10 -> Walts Power Supply Components:SO8-THERMAL
- U5: value TLV1117LV33 -> TLV1117LV33DCY
- moved C34 30.6 mm to (143.4, 11.4)
- moved FID2 23.0 mm to (126.9, 2.79)
- moved C14 16.2 mm to (146.4, 23.5), turned to 180 degrees
- moved FID3 14.6 mm to (40.3, 74.5)
- moved R16 13.6 mm to (135.7, 18.1), turned to 180 degrees
- moved D6 13.4 mm to (129.8, 21.6), turned to 180 degrees
- moved C2 13.4 mm to (44.5, 51.1)
- moved C1 12.6 mm to (45.2, 61.7), turned to 270 degrees
- moved C12 11.4 mm to (131.3, 40.4), turned to 270 degrees
- moved R17 11.3 mm to (135.7, 20.4), turned to 0 degrees
- moved C7 10.9 mm to (126.9, 36.2)
- moved C13 9.52 mm to (146.4, 25.9), turned to 180 degrees
- moved U3 7.51 mm to (129.4, 35.8), turned to 180 degrees
- moved R8 6.66 mm to (121.9, 24.1), turned to 90 degrees
- moved F1 6.65 mm to (127.8, 26.0)
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Connections:
- new net +3V3_HOMEPLUG: C16.1, J18.5, J18.6, J9.2, LED8.A, U5.2, U5.4
- net +3V3: now also C44.1, U12.5; no longer C16.1, J18.5, J18.6, J9.2, LED8.A, U5.2, U5.4
- net +5V: now also C43.1, L1.2, U12.1, U12.3; no longer L1.P$2, R13.2
- net ESC1_PWR: now also C39.+, J14.PWR1, J14.PWR2; no longer J14.1
- net ESC_1A: now also J14.A1, J14.A2; no longer J14.2
- net ESC_1B: now also J14.B1, J14.B2; no longer J14.3
- net ESC_1C: now also J14.C1, J14.C2; no longer J14.4
- net ESC_2A: now also J15.A1, J15.A2; no longer J15.2
- net ESC_2B: now also J15.B1, J15.B2; no longer J15.3
- net ESC_2C: now also J15.C1, J15.C2; no longer J15.4
- net ESC_3A: now also J16.A1, J16.A2; no longer J16.2
- net ESC_3B: now also J16.B1, J16.B2; no longer J16.3
- net ESC_3C: now also J16.C1, J16.C2; no longer J16.4
- net ESC_PWR2: now also C40.+, J15.PWR1, J15.PWR2; no longer J15.1
- net ESC_PWR3: now also C41.+, J16.PWR1, J16.PWR2; no longer J16.1
- net FUSED_VBAT: now also D6.C, R13.1, U4.2; no longer C10.1, R14.2, U4.1
- net GND: now also C39.-, C40.-, C41.-, C43.2, C44.2, D6.A, J14.GND1, J14.GND2, J15.GND1, J15.GND2, J16.GND1, J16.GND2, R14.1, U12.2, U4.4, U4.PAD; no longer C10.2, J14.5, J15.5, J16.5, R15.1, U4.11, U4.5, U4.7
- net N$16: now also U4.5; no longer U4.6
- net N$2: now also C42.2
- net N$20: now also R13.2, U4.7; no longer D6.A, R15.2, U4.8
- net N$23: now also U4.8; no longer U4.4
- net N$24: now also U4.1; no longer U4.10
- net N$25: now also L1.1, U4.3; no longer D6.C, L1.P$1, U4.9
- net N$27: now also C10.1, U4.6; no longer R14.1, U4.2
- net N$28: now also C10.2, R14.2; no longer R13.1, U4.3
- net N$7: now also C42.1
Routing:
- net +3V3_HOMEPLUG: track 0.00 -> 146.3 mm, vias 0 -> 3
- net +3V3: track 411.3 -> 280.5 mm, vias 9 -> 6
- net GND: track 321.2 -> 397.4 mm, vias 66 -> 75
- net FUSED_VBAT: track 18.4 -> 52.6 mm, vias 0 -> 8
- net N$24: track 7.83 -> 22.7 mm, vias 0 -> 2
- net 3V3_SCL: track 164.8 -> 152.7 mm
- net +5V: track 127.0 -> 135.5 mm, vias 32 -> 39
- net N$45: track 17.9 -> 25.1 mm
- net BAT_1+: track 60.8 -> 67.9 mm
- net BAT_1-1: track 76.5 -> 69.5 mm
- net ESC_3C: track 29.4 -> 35.6 mm
- net ESC_1A: track 9.44 -> 14.7 mm
- net ESC_2C: track 11.9 -> 17.2 mm
- net N$7: track 158.0 -> 152.8 mm
- net TETHER_B: track 193.1 -> 198.2 mm
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- added copper zone on layer 1, net +3V3_HOMEPLUG
- added copper zone on layer 1, net +5V
- added copper zone on layer 1, net ESC1_PWR
- added copper zone on layer 1, net ESC_PWR2
- added copper zone on layer 1, net ESC_PWR3
- added copper zone on layer 1, net GND
- added copper zone on layer 1, net N$25
Other:
- board text added: "Controller Board Rev 2.7"
- board text added: "Ext Svo Pwr"
- board text added: "HPWR HP ETH"
- board text removed: "Ext Servo Pwr"
- board text removed: "OpenROV Controller Board Rev 2.6"
- board text removed: "TPWR HP ETH"
- board text removed: "This work is released under the Creative Commons Attribution-NonCommercial-Share Alike 3.0 Unported License. All derivative works are to be attributed to OpenROV"
