File: OpenROV Controller.sch (EAGLE design)
At the start: 183 parts, among them J1 SSW-108-01-G-D, J18 SSW-103-01-G-D, J19 SSW-103-01-G-D, J2 SSW-108-01-G-D, J20 TSW-103-07-G-T, J21 TSW-103-07-G-T, J3 SSW-108-01-G-D, J4 SSW-108-01-G-D, J5 FCI 10090096-P254, J6 Samtec DW-23-11-G-D-630, Q1 SI4485, Q2 DMN65D8L, Q3 SI4425, Q4 IRLML6346TR, Q5 IRLML6346TR, Q6 IRLML6346TR, Q7 IRLML6346TR, Q8 FDV301N, Q9 FDV301N, U1 INA199A2, U10 INA199A2, U11 INA199A2, U2 INA199A2, U3 INA199A2, U4 LM25011, U5 TLV1117LV33, U6 ATMEGA2560-16AU, U7 TXB0108SSOP-20, U8 CAT24C256WI-G, U9 INA199A2, X1 16 MHz

Commit message: Checkin of the 2.7 schematics
Parts:
- removed R15: 0.075 1%, Walts_Generic_Parts:RESISTOR-1210
- added C39, C40, C41: 220 uF 35V Low-Impedance, Walts_Generic_Parts:CAP-POLARIZED-NICHICON-10MM
- added C42, C44: 1 uF 25V X7R, Walts_Generic_Parts:CAP0603
- added C43: 0.1 uF, Walts_Generic_Parts:CAP0603
- added U12: TCR2EF33, Walts Power Supply Components:TCR2EF
- C10: value 1 uF 50V X5R -> 3900 pF 25V NP0; device Walts_Generic_Parts:CAP0805 -> Walts_Generic_Parts:CAP0603
- C11: value 1000 pF 50V X7R -> 3900 pF 25V NP0
- C13, C14: value 10 uF 10V X5R -> 22 uF 10V X5R
- C16: value 10 uF 10V X5R -> 10 uF 25V X5R
- C34: value 220 uF 6.3V -> 220 uF 10V; device Walts_Generic_Parts:CAP-POLARIZED-B_CASE -> Walts_Generic_Parts:CAP-POLARIZED-NICHICON-8MM
- C35: value DNP -> 10 uF 25V X5R
- C8, C9: value 1 uF 50V X5R -> 10 uF 25V X5R
- D3: value SMAJ22A -> SMAJ18A
- D6: value CDBA340 -> SMAJ15A; device Walts_Generic_Parts:SCHOTTKYDO214AC -> Walts_Generic_Parts:ZENER-TVSDO-214AC
- F1: value 1.95A / 1.1A -> 2.0A / 4.0A 24V; device Walts_Generic_Parts:POLYFUSE-1812 -> Walts_Generic_Parts:POLYFUSE-2920
- J14: device OpenROV General Library:ESC_PADS-0.156_ALT -> OpenROV General Library:ESC_PADS-AFRO-12/20A-ESC1
- J15: device OpenROV General Library:ESC_PADS-0.156_ALT -> OpenROV General Library:ESC_PADS-AFRO-12/20A-ESC2
- J16: device OpenROV General Library:ESC_PADS-0.156_ALT -> OpenROV General Library:ESC_PADS-AFRO-12/20A-ESC3
- J18, J19: value SSW-103-01-G-D -> Sullins PRPC003DFAN-RC
- L1: value MSS1048-153MLB -> 15 uH 4A; device OpenROV Controller 2.5:INDUCTOR-MSS1048 -> Walts_Generic_Parts:INDUCTOR-BOURNS-12X0
- LED1, LED6: value Green -> GREEN
- LED7, LED8: value Yellow -> YELLOW
- Q3: value SI4425 -> SI4459ADY
- R13: value 10K -> 100K
- R14: value 133K 1% -> 13.0K 1%
- R16: value 9.76K 1% -> 45.3K 1%
- R24, R25, R26, R27, R28, R29, R30, R31, R32, R33, R34, R35: device Walts_Generic_Parts:RESISTOR-0603 -> Walts_Generic_Parts:RESISTOR-0805
- R67: value 0 -> 0 (Jumper)
- U4: value LM25011 -> Richtek RT8250; device OpenROV Controller 2.5:LM25011 -> Walts Power Supply Components:RICHTEK_82XX
- U5: value TLV1117LV33 -> TLV1117LV33DCY
Connections:
- new net +3V3_HOMEPLUG: C16.1, J18-5.1, J18-6.1, J9-2.S, LED8.A, U5.VOUT
- net +3V3: now also C44.1, U12.VOUT; no longer C16.1, J18-5.1, J18-6.1, J9-2.S, LED8.A, U5.VOUT
- net +5V: now also C43.1, U12.CTRL, U12.VIN; no longer R13.2
- net ESC1_PWR: now also C39.+
- net ESC_PWR2: now also C40.+
- net ESC_PWR3: now also C41.+
- net FUSED_VBAT: now also D6.C, R13.1; no longer C10.1, R14.2
- net GND: now also C39.-, C40.-, C41.-, C43.2, C44.2, D6.A, R14.1, U12.GND, U4.GND, U4.GNDPAD; no longer C10.2, R15.1, U4.CSG, U4.DAP, U4.SGND
- net N$2: now also C42.2
- net N$20: now also R13.2, U4.EN; no longer D6.A, R15.2, U4.CS
- net N$24: now also U4.BOOT; no longer U4.BST
- net N$25: no longer D6.C
- net N$27: now also C10.1, U4.COMP; no longer R14.1, U4.RT
- net N$28: now also C10.2, R14.2; no longer R13.1, U4.PGD
- net N$7: now also C42.1
Other:
- note added: "18 Aug 2014"
- note added: "2.7"
- note added: "30V 29A 5 mohm"
- note added: "For Battery outputs, 2.0A maximum current on each PWM channel For +5V outputs, maximum total PWM current is 1.5A For +3.3V outputs, maximum total PWM current is 0.2A"
- note added: "Header Pins for Tenda V2.0 Adapters 0.32" Engagement Length"
- note added: "HomePlug Adapter Power"
- note added: "OpenROV Controller 2.7"
- note added: "Revised ESC mounting pads to fit Afro 12A and 20A ESCs. New +5V switching power supply with 3A output vs. 1.6A on Controller 2.6. Resized programming resistors on power PWM outputs to handle 2A output vs 1A. Heavier traces on TP20-TP25. Revised ROV and ESC power switching. Additional +3.3V supply added to isolate homeplug adapter from +3.3V instrumentation"
- note removed: "+5V Supply Adapted from the CircuitCo OpenROV Cape"
- note removed: "30V 20A 10 mohm"
- note removed: "3A 40V"
- note removed: "Coilcraft Inductor 15 uH 0.04 ohm 3.5A"
- note removed: "OpenROV Controller 2.6"
- note removed: "Sockets for Tenda V2.0 Adapters"
- note removed: "Tether Power (HomePlug Adapter Power)"
- moved on the sheet: C10, C11, C12, C13, C15, C16, C34, C8, C9, D5, F1, R13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
